Commit message: now using only my local files for urdf

File: nuturtle_description/urdf/turtlebot3_burger.urdf (robot description, URDF)
Before this commit: robot turtlebot3_burger, 7 links, 6 joints
Links:
- link ${namespace}base_link: geometry collision box size=0.140 0.140 0.143; visual mesh filename=package://nuturtle_description/meshes/bases/burger_base.stl scale=0.001 0.001 0.001
- link ${namespace}base_scan: geometry collision cylinder length=0.0315 radius=0.055; visual mesh filename=package://nuturtle_description/meshes/sensors/lds.stl scale=0.001 0.001 0.001
- link ${namespace}wheel_left_link: geometry collision cylinder length=0.018 radius=0.033; visual mesh filename=package://nuturtle_description/meshes/wheels/left_tire.stl scale=0.001 0.001 0.001
- link ${namespace}wheel_right_link: geometry collision cylinder length=0.018 radius=0.033; visual mesh filename=package://nuturtle_description/meshes/wheels/right_tire.stl scale=0.001 0.001 0.001

Commit message: moved meshes to base mesh directory

File: nuturtle_description/urdf/turtlebot3_burger.urdf (robot description, URDF)
Before this commit: robot turtlebot3_burger, 7 links, 6 joints
Links:
- link ${namespace}base_link: geometry collision box size=0.140 0.140 0.143; visual mesh filename=package://nuturtle_description/meshes/burger_base.stl scale=0.001 0.001 0.001
- link ${namespace}base_scan: geometry collision cylinder length=0.0315 radius=0.055; visual mesh filename=package://nuturtle_description/meshes/lds.stl scale=0.001 0.001 0.001
- link ${namespace}wheel_left_link: geometry collision cylinder length=0.018 radius=0.033; visual mesh filename=package://nuturtle_description/meshes/left_tire.stl scale=0.001 0.001 0.001
- link ${namespace}wheel_right_link: geometry collision cylinder length=0.018 radius=0.033; visual mesh filename=package://nuturtle_description/meshes/right_tire.stl scale=0.001 0.001 0.001
