Commit message: parametrizing xacro. done all except wheel spacing

File: nuturtle_description/urdf/turtlebot3_burger.urdf.xacro (robot description, xacro)
@@ -6,4 +6,6 @@
   <xacro:arg name="namespace" default=""/>
   <xacro:property name="namespace" value="$(arg namespace)"/>
+  <xacro:property name="yaml_file" value="$(find nuturtle_description)/config/diff_params.yaml"/>
+  <xacro:property name="props" value="${xacro.load_yaml(yaml_file)['/**']['ros__parameters']}"/>
   <!-- Init colour -->
   <material name="black">
@@ -54,5 +56,5 @@
       <origin xyz="-0.032 0 0.070" rpy="0 0 0"/>
       <geometry>
-        <box size="0.140 0.140 0.143"/>
+        <cylinder length="0.143" radius="${props['collision_radius']}"/>
       </geometry>
     </collision>
@@ -80,5 +82,5 @@
       <origin xyz="0 0 0" rpy="0 0 0"/>
       <geometry>
-        <cylinder length="0.018" radius="0.033"/>
+        <cylinder length="0.018" radius="${props['wheel_radius']}"/>
       </geometry>
     </collision>
@@ -106,5 +108,5 @@
       <origin xyz="0 0 0" rpy="0 0 0"/>
       <geometry>
-        <cylinder length="0.018" radius="0.033"/>
+        <cylinder length="0.018" radius="${props['wheel_radius']}"/>
       </geometry>
     </collision>

Commit message: parametrized track width

File: nuturtle_description/urdf/turtlebot3_burger.urdf.xacro (robot description, xacro)
@@ -68,5 +68,5 @@
     <parent link="${namespace}base_link"/>
     <child link="${namespace}wheel_left_link"/>
-    <origin xyz="0.0 0.08 0.023" rpy="-1.57 0 0"/>
+    <origin xyz="0.0 ${props['track_width']/2} 0.023" rpy="-1.57 0 0"/>
     <axis xyz="0 0 1"/>
   </joint>
@@ -94,5 +94,5 @@
     <parent link="${namespace}base_link"/>
     <child link="${namespace}wheel_right_link"/>
-    <origin xyz="0.0 -0.080 0.023" rpy="-1.57 0 0"/>
+    <origin xyz="0.0 -${props['track_width']/2} 0.023" rpy="-1.57 0 0"/>
     <axis xyz="0 0 1"/>
   </joint>

Commit message: added color to urdf. defaulting to purple

File: nuturtle_description/urdf/turtlebot3_burger.urdf.xacro (robot description, xacro)
@@ -5,4 +5,6 @@
   xmlns:xacro="http://ros.org/wiki/xacro">
   <xacro:arg name="namespace" default=""/>
+  <xacro:arg name="color" default="purple"/>
+  <xacro:property name="color" value="$(arg color)"/>
   <xacro:property name="namespace" value="$(arg namespace)"/>
   <xacro:property name="yaml_file" value="$(find nuturtle_description)/config/diff_params.yaml"/>
@@ -39,4 +41,7 @@
     <color rgba="1.0 1.0 1.0 1.0"/>
   </material>
+  <material name="purple">
+    <color rgba="0.3 0.16 0.52 1.0"/>
+  </material>
   <link name="${namespace}base_footprint"/>
   <joint name="${namespace}base_joint" type="fixed">
@@ -51,5 +56,5 @@
         <mesh filename="package://nuturtle_description/meshes/burger_base.stl" scale="0.001 0.001 0.001"/>
       </geometry>
-      <material name="light_black"/>
+      <material name="${color}"/>
     </visual>
     <collision>

Commit message: now supporting purple robot!

File: nuturtle_description/urdf/turtlebot3_burger.urdf.xacro (robot description, xacro)
@@ -7,5 +7,5 @@
   <xacro:arg name="color" default="purple"/>
   <xacro:property name="color" value="$(arg color)"/>
-  <xacro:property name="namespace" value="$(arg namespace)"/>
+  <xacro:property name="namespace" value="$(arg color)_"/>
   <xacro:property name="yaml_file" value="$(find nuturtle_description)/config/diff_params.yaml"/>
   <xacro:property name="props" value="${xacro.load_yaml(yaml_file)['/**']['ros__parameters']}"/>

Commit message: fixed tf prefix issue in nuturtle_description.
now need to fix the rviz files over there

File: nuturtle_description/urdf/turtlebot3_burger.urdf.xacro (robot description, xacro)
@@ -7,5 +7,5 @@
   <xacro:arg name="color" default="purple"/>
   <xacro:property name="color" value="$(arg color)"/>
-  <xacro:property name="namespace" value="$(arg color)_"/>
+  <xacro:property name="namespace" value="$(arg namespace)"/>
   <xacro:property name="yaml_file" value="$(find nuturtle_description)/config/diff_params.yaml"/>
   <xacro:property name="props" value="${xacro.load_yaml(yaml_file)['/**']['ros__parameters']}"/>
